Commit message: first initial commit after changes

File: ros2_ws/src/space_description/urdf/space_rover.urdf.xacro (robot description, xacro)
@@ -1,5 +1,4 @@
 <?xml version="1.0"?>
 <robot name="space_rover" xmlns:xacro="http://ros.org/wiki/xacro">
-  <xacro:arg name="use_sim" default="true"/>
   <xacro:property name="base_length" value="0.32"/>
   <xacro:property name="base_width" value="0.26"/>
@@ -79,4 +78,11 @@
     <origin xyz="0.17 0 0.07" rpy="0 0 0"/>
   </joint>
+  <!-- REP-103 optical coordinates: Z forward, X right, Y down. -->
+  <link name="camera_optical_frame"/>
+  <joint name="camera_optical_joint" type="fixed">
+    <parent link="camera_link"/>
+    <child link="camera_optical_frame"/>
+    <origin xyz="0 0 0" rpy="-1.57079632679 0 -1.57079632679"/>
+  </joint>
   <link name="imu_link">
     <inertial>
@@ -90,4 +96,3 @@
     <origin xyz="0 0 0.03" rpy="0 0 0"/>
   </joint>
-  <xacro:include filename="$(find space_description)/urdf/gazebo.xacro"/>
 </robot>

File: ros2_ws/src/space_gazebo/urdf/gazebo_extensions.xacro (robot description, xacro)
@@ -13,11 +13,15 @@
     <plugin filename="gz-sim-diff-drive-system"
             name="gz::sim::systems::DiffDrive">
+      <!--
+        Temporary Phase 1 backend only. Milestone A replaces direct ROS
+        authority with ArduPilot Rover SITL and the ArduPilot Gazebo plugin.
+      -->
       <left_joint>left_front_wheel_joint</left_joint>
       <left_joint>left_rear_wheel_joint</left_joint>
       <right_joint>right_front_wheel_joint</right_joint>
       <right_joint>right_rear_wheel_joint</right_joint>
-      <wheel_separation>0.35</wheel_separation>
-      <wheel_radius>0.112</wheel_radius>
-      <topic>/cmd_vel</topic>
+      <wheel_separation>${2 * wheel_y}</wheel_separation>
+      <wheel_radius>${wheel_radius}</wheel_radius>
+      <topic>/cmd_vel_safe</topic>
     </plugin>
   </gazebo>
@@ -26,4 +30,5 @@
             name="gz::sim::systems::OdometryPublisher">
       <odom_publish_frequency>50</odom_publish_frequency>
+      <dimensions>3</dimensions>
       <odom_frame>odom</odom_frame>
       <robot_base_frame>base_footprint</robot_base_frame>
@@ -41,4 +46,5 @@
   <gazebo reference="camera_link">
     <sensor name="front_rgbd" type="rgbd">
+      <!-- Gazebo RGBD point coordinates are X-forward in camera_link. -->
       <gz_frame_id>camera_link</gz_frame_id>
       <update_rate>15</update_rate>

Commit message: stl file upload + integration into urdf xacro file

File: ros2_ws/src/space_description/urdf/space_rover.urdf.xacro (robot description, xacro)
@@ -1,4 +1,20 @@
 <?xml version="1.0"?>
 <robot name="space_rover" xmlns:xacro="http://ros.org/wiki/xacro">
+  <!--
+    Complete CAD visual controls. The STL is exported in millimetres and uses
+    -X as forward, so the default transform scales, centers, and rotates it
+    into the base_link REP-103 frame. Override these xacro arguments when
+    refining alignment without editing individual link visuals.
+  -->
+  <xacro:arg name="use_rover_stl_visual" default="true"/>
+  <xacro:arg name="rover_mesh_scale" default="0.001 0.001 0.001"/>
+  <xacro:arg name="rover_mesh_xyz" default="0.00875 0 -0.09269867"/>
+  <xacro:arg name="rover_mesh_rpy" default="0 0 3.14159265359"/>
+  <xacro:property
+    name="use_rover_stl_visual"
+    value="$(arg use_rover_stl_visual)"/>
+  <xacro:property name="rover_mesh_scale" value="$(arg rover_mesh_scale)"/>
+  <xacro:property name="rover_mesh_xyz" value="$(arg rover_mesh_xyz)"/>
+  <xacro:property name="rover_mesh_rpy" value="$(arg rover_mesh_rpy)"/>
   <xacro:property name="base_length" value="0.32"/>
   <xacro:property name="base_width" value="0.26"/>
@@ -19,8 +35,21 @@
   </joint>
   <link name="base_link">
-    <visual>
-      <geometry><box size="${base_length} ${base_width} ${base_height}"/></geometry>
-      <material name="chassis_dark"/>
-    </visual>
+    <xacro:if value="${use_rover_stl_visual}">
+      <visual name="rover_complete_stl_visual">
+        <origin xyz="${rover_mesh_xyz}" rpy="${rover_mesh_rpy}"/>
+        <geometry>
+          <mesh
+            filename="package://space_description/meshes/rover/rover_prototype.stl"
+            scale="${rover_mesh_scale}"/>
+        </geometry>
+        <material name="chassis_dark"/>
+      </visual>
+    </xacro:if>
+    <xacro:unless value="${use_rover_stl_visual}">
+      <visual name="primitive_chassis_visual">
+        <geometry><box size="${base_length} ${base_width} ${base_height}"/></geometry>
+        <material name="chassis_dark"/>
+      </visual>
+    </xacro:unless>
     <collision>
       <geometry><box size="${base_length} ${base_width} ${base_height}"/></geometry>
@@ -34,9 +63,11 @@
   <xacro:macro name="wheel" params="prefix x y">
     <link name="${prefix}_wheel">
-      <visual>
-        <origin xyz="0 0 0" rpy="1.57079632679 0 0"/>
-        <geometry><cylinder radius="${wheel_radius}" length="${wheel_width}"/></geometry>
-        <material name="wheel_gray"/>
-      </visual>
+      <xacro:unless value="${use_rover_stl_visual}">
+        <visual name="${prefix}_primitive_wheel_visual">
+          <origin xyz="0 0 0" rpy="1.57079632679 0 0"/>
+          <geometry><cylinder radius="${wheel_radius}" length="${wheel_width}"/></geometry>
+          <material name="wheel_gray"/>
+        </visual>
+      </xacro:unless>
       <collision>
         <origin xyz="0 0 0" rpy="1.57079632679 0 0"/>

Commit message: urdf skrt~~~

File: ros2_ws/src/space_description/urdf/space_rover.urdf.xacro (robot description, xacro)
@@ -20,9 +20,11 @@
   <xacro:property name="base_width" value="0.26"/>
   <xacro:property name="base_height" value="0.10"/>
-  <xacro:property name="wheel_radius" value="0.112"/>
-  <xacro:property name="wheel_width" value="0.045"/>
-  <xacro:property name="wheel_x" value="0.145"/>
-  <xacro:property name="wheel_y" value="0.175"/>
-  <xacro:property name="wheel_z" value="0.02"/>
+  <!-- Dimensions and axle centers measured from the complete CAD STL. -->
+  <xacro:property name="wheel_radius" value="0.070"/>
+  <xacro:property name="wheel_width" value="0.040"/>
+  <xacro:property name="front_wheel_x" value="0.08375"/>
+  <xacro:property name="rear_wheel_x" value="-0.06625"/>
+  <xacro:property name="wheel_y" value="0.11650"/>
+  <xacro:property name="wheel_z" value="-0.06400"/>
   <material name="chassis_dark"><color rgba="0.10 0.12 0.14 1.0"/></material>
   <material name="wheel_gray"><color rgba="0.35 0.38 0.40 1.0"/></material>
@@ -32,5 +34,5 @@
     <parent link="base_footprint"/>
     <child link="base_link"/>
-    <origin xyz="0 0 ${wheel_radius + base_height * 0.5 - 0.025}" rpy="0 0 0"/>
+    <origin xyz="0 0 ${wheel_radius - wheel_z}" rpy="0 0 0"/>
   </joint>
   <link name="base_link">
@@ -61,6 +63,19 @@
     </inertial>
   </link>
-  <xacro:macro name="wheel" params="prefix x y">
+  <xacro:macro name="wheel" params="prefix x y mesh_file">
     <link name="${prefix}_wheel">
+      <xacro:if value="${use_rover_stl_visual}">
+        <visual name="${prefix}_cad_wheel_visual">
+          <!-- Centered wheel STL uses the same millimetre scale and -X-forward
+               CAD orientation as the complete rover assembly. -->
+          <origin xyz="0 0 0" rpy="0 0 3.14159265359"/>
+          <geometry>
+            <mesh
+              filename="package://space_description/meshes/rover/${mesh_file}"
+              scale="${rover_mesh_scale}"/>
+          </geometry>
+          <material name="wheel_gray"/>
+        </visual>
+      </xacro:if>
       <xacro:unless value="${use_rover_stl_visual}">
         <visual name="${prefix}_primitive_wheel_visual">
@@ -83,12 +98,28 @@
       <parent link="base_link"/>
       <child link="${prefix}_wheel"/>
-      <origin xyz="${x} ${y} ${wheel_z - base_height * 0.5}" rpy="0 0 0"/>
+      <origin xyz="${x} ${y} ${wheel_z}" rpy="0 0 0"/>
       <axis xyz="0 1 0"/>
     </joint>
   </xacro:macro>
-  <xacro:wheel prefix="left_front" x="${wheel_x}" y="${wheel_y}"/>
-  <xacro:wheel prefix="left_rear" x="-${wheel_x}" y="${wheel_y}"/>
-  <xacro:wheel prefix="right_front" x="${wheel_x}" y="-${wheel_y}"/>
-  <xacro:wheel prefix="right_rear" x="-${wheel_x}" y="-${wheel_y}"/>
+  <xacro:wheel
+    prefix="left_front"
+    x="${front_wheel_x}"
+    y="${wheel_y}"
+    mesh_file="left_front_wheel.stl"/>
+  <xacro:wheel
+    prefix="left_rear"
+    x="${rear_wheel_x}"
+    y="${wheel_y}"
+    mesh_file="left_rear_wheel.stl"/>
+  <xacro:wheel
+    prefix="right_front"
+    x="${front_wheel_x}"
+    y="-${wheel_y}"
+    mesh_file="right_front_wheel.stl"/>
+  <xacro:wheel
+    prefix="right_rear"
+    x="${rear_wheel_x}"
+    y="-${wheel_y}"
+    mesh_file="right_rear_wheel.stl"/>
   <link name="camera_link">
     <visual>

Commit message: Make rover geometry a single source of truth
One CAD import (51b34ac, wheel radius 0.112 -> 0.070 m) invalidated four
values across four packages, and every one failed silently because the
arithmetic downstream still succeeded and the outputs still looked
plausible. Copying a CAD number into a config is what created each one,
so config/rover_geometry.yaml now holds the measured primitives and
nothing derivable is stored anywhere.

- rover_geometry.py derives the step limit, wheel separation, track
  width, wheelbase, base_link height, nav2 footprint, and minimum
  passable width. It ships here, beside the geometry it reads, because
  this package owns the physical description and depends on nothing --
  perception, bringup, and mission can all import it without inverting
  the dependency graph. Putting the source in space_mission, the literal
  reading of "the RoverSpec YAML is the source", would have made
  space_description depend on the mission layer to build its own URDF.
- space_rover.urdf.xacro consumes it via xacro.load_yaml instead of
  declaring its own copies. Generated URDF is byte-identical to before,
  confirming the wiring changed no number.
- Missing keys raise instead of defaulting: a silently defaulted
  dimension is the failure this exists to prevent.

Two measured values are recorded that are NOT derivable, with how they
were obtained:

- chassis_ground_clearance is 0.030 m from a vertex sweep of
  rover_prototype.stl, not the 0.084 m the collision box implies. The
  hub and motor bosses that reach below the contact plane are excluded
  by name and count, since the tyre meets terrain there first.
- mass_base + 4*mass_wheel = 2.36 kg does not match the 3.0 kg in
  CLAUDE.md. Recorded rather than reconciled: agreeing them changes sim
  dynamics, so that is its own change.

test_rover_geometry.py exists to make the NEXT CAD change loud. It
asserts the step limit is half the wheel radius, that wheel contact
lands exactly on base_footprint for any wheel size, that the footprint
covers both the collision box and the wheels, and that the recorded
wheel still matches left_front_wheel.stl. Verified by temporarily
setting wheel_radius to 0.100: derived values, the URDF, and the
footprint all followed, and the STL check failed as intended.

Uses explicit ament_flake8/ament_pep257 rather than ament_lint_auto,
matching space_perception: lint_auto adds ament_copyright, and no Python
file in this workspace carries a copyright header. Tests: 19, 0 failures.

File: ros2_ws/src/space_description/urdf/space_rover.urdf.xacro (robot description, xacro)
@@ -17,14 +17,25 @@
   <xacro:property name="rover_mesh_xyz" value="$(arg rover_mesh_xyz)"/>
   <xacro:property name="rover_mesh_rpy" value="$(arg rover_mesh_rpy)"/>
-  <xacro:property name="base_length" value="0.32"/>
-  <xacro:property name="base_width" value="0.26"/>
-  <xacro:property name="base_height" value="0.10"/>
-  <!-- Dimensions and axle centers measured from the complete CAD STL. -->
-  <xacro:property name="wheel_radius" value="0.070"/>
-  <xacro:property name="wheel_width" value="0.040"/>
-  <xacro:property name="front_wheel_x" value="0.08375"/>
-  <xacro:property name="rear_wheel_x" value="-0.06625"/>
-  <xacro:property name="wheel_y" value="0.11650"/>
-  <xacro:property name="wheel_z" value="-0.06400"/>
+  <!--
+    Dimensions come from config/rover_geometry.yaml, the single source of truth,
+    and are NOT written here. The last CAD import silently invalidated four
+    values across four packages because each had its own copy of the wheel
+    radius; this file consumes the source instead of duplicating it. To change a
+    dimension, edit that YAML.
+  -->
+  <xacro:property
+    name="geom"
+    value="${xacro.load_yaml('$(find space_description)/config/rover_geometry.yaml')}"/>
+  <xacro:property name="base_length" value="${geom['base_length']}"/>
+  <xacro:property name="base_width" value="${geom['base_width']}"/>
+  <xacro:property name="base_height" value="${geom['base_height']}"/>
+  <xacro:property name="wheel_radius" value="${geom['wheel_radius']}"/>
+  <xacro:property name="wheel_width" value="${geom['wheel_width']}"/>
+  <xacro:property name="front_wheel_x" value="${geom['front_wheel_x']}"/>
+  <xacro:property name="rear_wheel_x" value="${geom['rear_wheel_x']}"/>
+  <xacro:property name="wheel_y" value="${geom['wheel_y']}"/>
+  <xacro:property name="wheel_z" value="${geom['wheel_z']}"/>
+  <xacro:property name="mass_base" value="${geom['mass_base']}"/>
+  <xacro:property name="mass_wheel" value="${geom['mass_wheel']}"/>
   <material name="chassis_dark"><color rgba="0.10 0.12 0.14 1.0"/></material>
   <material name="wheel_gray"><color rgba="0.35 0.38 0.40 1.0"/></material>
@@ -58,5 +69,5 @@
     </collision>
     <inertial>
-      <mass value="1.8"/>
+      <mass value="${mass_base}"/>
       <origin xyz="0 0 0" rpy="0 0 0"/>
       <inertia ixx="0.018" ixy="0" ixz="0" iyy="0.022" iyz="0" izz="0.030"/>
@@ -90,5 +101,5 @@
       </collision>
       <inertial>
-        <mass value="0.14"/>
+        <mass value="${mass_wheel}"/>
         <origin xyz="0 0 0" rpy="0 0 0"/>
         <inertia ixx="0.00045" ixy="0" ixz="0" iyy="0.00045" iyz="0" izz="0.00045"/>

Commit message: Correct the simulated mass and fit the collision box to the CAD
Two geometry defects, both in the direction that flatters the rover.

MASS. Three different numbers were in play: 3.000 kg (competition ceiling),
2.725 kg (design estimate, master document), and 2.450 kg (what the URDF
actually summed to -- 1.8 base + 4x0.14 wheels + 0.08 camera + 0.01 IMU).
The sim was 10.1% light. For this mission that is not cosmetic: slip is the
signature measurement, and a rover that is too light slips less, climbs
better, and finds more traction than the real one, so a validation run on
it validates nothing.

mass_total is now the authority at 2.725 kg and mass_base is DERIVED as the
remainder, because the chassis is the least-known component while the total
is the constrained one -- letting the parts define the total is how they
drifted apart. base_link inertia became a per-kilogram triple so it scales
with the derived mass instead of describing the old 1.8 kg chassis forever.
mass_limit records 3.0 kg as the ceiling it is, and a test asserts the
design estimate stays under it. The generated URDF now sums to exactly
2.725000 kg, checked by parsing xacro output rather than the derivation.

CLAUDE.md said "3 kg" without qualification, which is what let the ceiling
be used as a design value; it now states both numbers and which is which.
ground_pressure_kpa was 3.47, computed from the ceiling -- it is derived
now, giving 3.157.

COLLISION BOX. The 0.32 x 0.26 x 0.10 box was wrong in both directions:
15 mm longer than the real chassis and 13 mm NARROWER. Over-size is merely
conservative; under-size lets Gazebo pass the rover through gaps it would
physically hit, and judging passable gaps is part of the mission. The box is
now derived from measured mesh extents (0.30521 x 0.27300 x 0.16405) with an
explicit origin, since the chassis is not centred on base_link.

It spans clearance-to-top rather than the full mesh bbox on purpose: the mesh
dips 8 mm below the contact plane at the wheel hubs, and a box that deep
would rest the rover on its chassis instead of its wheels. An axis-aligned
box cannot represent this chassis exactly -- see docs/pending.md.

The shorter box moves the nav2 footprint from 0.16 to 0.15375 in x, which the
footprint guard test caught rather than letting drift.

Tests: space_description 26, space_bringup 9, 0 failures.

File: ros2_ws/src/space_description/urdf/space_rover.urdf.xacro (robot description, xacro)
@@ -27,7 +27,4 @@
     name="geom"
     value="${xacro.load_yaml('$(find space_description)/config/rover_geometry.yaml')}"/>
-  <xacro:property name="base_length" value="${geom['base_length']}"/>
-  <xacro:property name="base_width" value="${geom['base_width']}"/>
-  <xacro:property name="base_height" value="${geom['base_height']}"/>
   <xacro:property name="wheel_radius" value="${geom['wheel_radius']}"/>
   <xacro:property name="wheel_width" value="${geom['wheel_width']}"/>
@@ -36,6 +33,44 @@
   <xacro:property name="wheel_y" value="${geom['wheel_y']}"/>
   <xacro:property name="wheel_z" value="${geom['wheel_z']}"/>
-  <xacro:property name="mass_base" value="${geom['mass_base']}"/>
+  <!--
+    Chassis collision box, derived from the measured mesh extents. It replaces a
+    0.32 x 0.26 x 0.10 box that was 15 mm too long and 13 mm too NARROW.
+    Over-size is merely conservative; under-size lets Gazebo pass the rover
+    through gaps it would physically hit. Vertically it spans the measured
+    ground clearance to the chassis top rather than the full mesh bbox, because
+    the mesh dips 8 mm below the contact plane at the wheel hubs and a box that
+    deep would rest the rover on its chassis instead of its wheels.
+  -->
+  <xacro:property name="chassis_box_length"
+    value="${geom['chassis_max_x'] - geom['chassis_min_x']}"/>
+  <xacro:property name="chassis_box_width"
+    value="${2 * geom['chassis_half_y']}"/>
+  <xacro:property name="chassis_box_height"
+    value="${geom['chassis_top_z'] - geom['chassis_ground_clearance']}"/>
+  <xacro:property name="chassis_box_x"
+    value="${(geom['chassis_min_x'] + geom['chassis_max_x']) / 2}"/>
+  <!-- base_link sits wheel_radius - wheel_z above the contact plane. -->
+  <xacro:property name="chassis_box_z"
+    value="${(geom['chassis_ground_clearance'] + geom['chassis_top_z']) / 2
+             - (geom['wheel_radius'] - geom['wheel_z'])}"/>
+  <!--
+    mass_base is the REMAINDER of mass_total after the wheels, camera, and IMU,
+    so the parts can never drift from the total the way they did before: the URDF
+    summed to 2.450 kg against a 2.725 kg design estimate. Inertia scales with
+    that derived mass instead of being a fixed triple describing the old 1.8 kg
+    chassis.
+  -->
   <xacro:property name="mass_wheel" value="${geom['mass_wheel']}"/>
+  <xacro:property name="mass_camera" value="${geom['mass_camera']}"/>
+  <xacro:property name="mass_imu" value="${geom['mass_imu']}"/>
+  <xacro:property name="mass_base"
+    value="${geom['mass_total'] - 4 * geom['mass_wheel']
+             - geom['mass_camera'] - geom['mass_imu']}"/>
+  <xacro:property name="base_ixx"
+    value="${geom['base_inertia_per_kg']['ixx'] * mass_base}"/>
+  <xacro:property name="base_iyy"
+    value="${geom['base_inertia_per_kg']['iyy'] * mass_base}"/>
+  <xacro:property name="base_izz"
+    value="${geom['base_inertia_per_kg']['izz'] * mass_base}"/>
   <material name="chassis_dark"><color rgba="0.10 0.12 0.14 1.0"/></material>
   <material name="wheel_gray"><color rgba="0.35 0.38 0.40 1.0"/></material>
@@ -61,15 +96,22 @@
     <xacro:unless value="${use_rover_stl_visual}">
       <visual name="primitive_chassis_visual">
-        <geometry><box size="${base_length} ${base_width} ${base_height}"/></geometry>
+        <origin xyz="${chassis_box_x} 0 ${chassis_box_z}" rpy="0 0 0"/>
+        <geometry>
+          <box size="${chassis_box_length} ${chassis_box_width} ${chassis_box_height}"/>
+        </geometry>
         <material name="chassis_dark"/>
       </visual>
     </xacro:unless>
     <collision>
-      <geometry><box size="${base_length} ${base_width} ${base_height}"/></geometry>
+      <origin xyz="${chassis_box_x} 0 ${chassis_box_z}" rpy="0 0 0"/>
+      <geometry>
+        <box size="${chassis_box_length} ${chassis_box_width} ${chassis_box_height}"/>
+      </geometry>
     </collision>
     <inertial>
       <mass value="${mass_base}"/>
       <origin xyz="0 0 0" rpy="0 0 0"/>
-      <inertia ixx="0.018" ixy="0" ixz="0" iyy="0.022" iyz="0" izz="0.030"/>
+      <inertia ixx="${base_ixx}" ixy="0" ixz="0" iyy="${base_iyy}" iyz="0"
+        izz="${base_izz}"/>
     </inertial>
   </link>
@@ -142,5 +184,5 @@
     </collision>
     <inertial>
-      <mass value="0.08"/>
+      <mass value="${mass_camera}"/>
       <inertia ixx="0.00002" ixy="0" ixz="0" iyy="0.00002" iyz="0" izz="0.00002"/>
     </inertial>
@@ -160,5 +202,5 @@
   <link name="imu_link">
     <inertial>
-      <mass value="0.01"/>
+      <mass value="${mass_imu}"/>
       <inertia ixx="0.000001" ixy="0" ixz="0" iyy="0.000001" iyz="0" izz="0.000001"/>
     </inertial>
