Commit message: Survey the whole arena, and fix the review findings it depended on
MAP. survey_arena.py places the rover at 96 poses (4x6 grid, 4 yaws) and
lets the pipeline observe from each, giving 75.0% coverage of the arena --
6000 of 8000 cells, median 29 visits each -- against 8.7% from a driven
run. Crater floors read green and rims dark red, matching the structure
the CAD hillshade shows independently.

Placement is not a shortcut around a bug: this rover genuinely cannot
traverse the arena, it high-centres on the rims at 1.1 m. Perception is
fully exercised (real rendered depth through the unchanged pipeline);
only locomotion is skipped, and the figure title and README both say so.
Placement heights come from the CAD grid so the rover settles onto the
surface rather than being dropped inside it; 21 of 96 poses still ended
tilted past 25 deg and that is reported, not hidden. The odom trace is
deliberately NOT drawn in survey mode -- it is a sequence of teleports and
would read as a route the rover cannot actually drive.

Validation over the full survey, 157378 cells: correlation +0.707, error
sd 6.78 deg, median -2.76 deg. The bias sign is unchanged and is the
point: perception UNDER-reports slope, so a geometry-only map flatters the
terrain, which is the quantified case for measuring slip on top of it.

REVIEW FINDINGS. The footprint one was a real safety defect I introduced:
footprint_half_extents unioned the chassis box and wheels but omitted
camera_link's collision box, which reaches 0.1975 m forward -- 43.8 mm
beyond the footprint both costmaps were then shrunk to. A footprint
smaller than what Gazebo collides with lets nav2 plan the rover into
contact.

Worth recording WHY the guard test missed it: it asserted the footprint
covered the chassis and the wheels, i.e. exactly the two shapes the
derivation considered, so it inherited the blind spot instead of catching
it. It is replaced by test_footprint_covers_every_collision, which walks
the generated URDF and checks every collision element, so a link added
later fails even if nobody updates the derivation. That test caught the
stale nav2 literal immediately after the fix.

Also fixed:
- wheel_linear_speed returned a one-sided average when a side's joints
  were missing -- the speed of a turning rover reported as straight-line
  travel, flowing into slip as a valid reading. It now returns None and
  the node warns once. An existing test had frozen the defect into the
  contract by asserting the one-sided result; it now asserts the opposite.
- _slip_ema survived input dropouts and blended pre-outage slip into the
  first readings after recovery, which is when the terrain is most likely
  to have changed. Reset on both stale and uncomputable paths.
- a NaN or negative twist covariance mapped to quality 1.0, so "covariance
  unknown" was reported as fully trusted. Now 0.0; exactly zero still
  means 1.0, which is Gazebo ground truth saying the pose IS exact.
- slip.yaml and the node default still hard-copied wheel_radius 0.070,
  the very duplication this branch exists to remove. Derived now, and
  absent from the YAML so there is one source.
- max_step_height_m is capped by ground_clearance_m: the wheel-derived
  0.035 m exceeded the measured 0.030 m clearance, so traversability would
  have called a step climbable that grounds the chassis first. For the
  medium rover the wheel still binds, so the cap is not one-sided.
- space_mission never declared space_msgs (imported since the last commit)
  or numpy, and space_perception declared space_description only as
  exec_depend although traversability_calibration imports it at module
  level. Both fail in a clean workspace and pass in a warm one.
- rover_spec_small.yaml still re-types four values the geometry source
  owns, which gave two independent sources for one step limit. The copies
  stay -- deleting them would stop the mission layer reading a spec
  without a sourced workspace -- but a test now binds them to the source.

Tests: 185, 0 failures across the five active packages.

File: ros2_ws/src/space_description/urdf/space_rover.urdf.xacro (robot description, xacro)
@@ -62,4 +62,7 @@
   -->
   <xacro:property name="mass_wheel" value="${geom['mass_wheel']}"/>
+  <xacro:property name="camera_mount_x" value="${geom['camera_mount_x']}"/>
+  <xacro:property name="camera_box_l" value="${geom['camera_collision_length']}"/>
+  <xacro:property name="camera_box_w" value="${geom['camera_collision_width']}"/>
   <xacro:property name="mass_camera" value="${geom['mass_camera']}"/>
   <xacro:property name="mass_imu" value="${geom['mass_imu']}"/>
@@ -177,9 +180,9 @@
   <link name="camera_link">
     <visual>
-      <geometry><box size="0.055 0.025 0.025"/></geometry>
+      <geometry><box size="${camera_box_l} ${camera_box_w} 0.025"/></geometry>
       <material name="camera_blue"/>
     </visual>
     <collision>
-      <geometry><box size="0.055 0.025 0.025"/></geometry>
+      <geometry><box size="${camera_box_l} ${camera_box_w} 0.025"/></geometry>
     </collision>
     <inertial>
@@ -191,5 +194,5 @@
     <parent link="base_link"/>
     <child link="camera_link"/>
-    <origin xyz="0.17 0 0.07" rpy="0 0 0"/>
+    <origin xyz="${camera_mount_x} 0 0.07" rpy="0 0 0"/>
   </joint>
   <!-- REP-103 optical coordinates: Z forward, X right, Y down. -->
