Commit message: fix: correct wheel radius and re-pin SITL to the flashed firmware
The physical rover's wheels were changed from 140 mm to 120 mm diameter and
the URDF was never updated, so wheel_radius was overstating every distance
derived from it by about 17%. Set it from the build rather than the CAD.

Record what is still unreconciled rather than quietly picking a number. The
visual mesh still shows 140 mm wheels, and wheel_y remains the CAD value,
which disagrees with a tape measurement of the physical track width. Both
are noted in the URDF so that anything converting wheel counts to distance
uses the build values knowingly.

Re-pin SITL from Rover-4.6.3 to Rover-4.7.0 to match the firmware actually
flashed on the Pixhawk 6X, and note that 4.7 and later require the v4.7.0
branch of Micro-XRCE-DDS-Gen rather than v4.5.1.

The DDS interface measurements already recorded were taken on 4.6.3. They
are marked as not yet repeated on 4.7.0 instead of being carried over, since
AP_DDS publisher and topic behaviour can change between releases.

Also record what the connected board reports: firmware 4.7.0 with no
DDS_ENABLE parameter, so the flashed build contains no AP_DDS and the
hardware transport question stays open.

Co-Authored-By: Claude Opus 5 (1M context) <noreply@anthropic.com>

File: ros2_ws/src/space_description/urdf/space_rover.urdf.xacro (robot description, xacro)
@@ -20,6 +20,12 @@
   <xacro:property name="base_width" value="0.26"/>
   <xacro:property name="base_height" value="0.10"/>
-  <!-- Dimensions and axle centers measured from the complete CAD STL. -->
-  <xacro:property name="wheel_radius" value="0.070"/>
+  <!-- Axle centers measured from the complete CAD STL.
+       wheel_radius is NOT from that CAD: the wheels were changed from 140 mm
+       to 120 mm diameter on the physical rover, so it is set from the build
+       rather than the model. The visual mesh still shows the 140 mm wheels.
+       wheel_y is still the CAD value and disagrees with a tape measurement of
+       the physical track width; it has not been reconciled yet. Anything that
+       converts wheel counts to distance must use these values, not the CAD. -->
+  <xacro:property name="wheel_radius" value="0.060"/>
   <xacro:property name="wheel_width" value="0.040"/>
   <xacro:property name="front_wheel_x" value="0.08375"/>

Commit message: fix(description): use the measured track width, not the CAD value
The rover's track width measures 225 mm centre to centre; the URDF carried
the CAD's 233 mm. Wheel radius was already corrected to the built 60 mm.
Both now come from the rover rather than the model, because everything that
turns wheel counts into motion depends on them: the radius scales distance
and the track width scales every turn, so a 3.4% track error is roughly 12
degrees of heading error per full rotation.

With both measured, the odometry constants are pinned:

  wheel circumference 0.37699 m, 6400 counts per output revolution
  metres per count    5.8905e-5
  v_wheel             counts_per_sec * 5.8905e-5
  omega               (v_right - v_left) / 0.225

This also corrects a constant that was in use for slip calculations. It read
0.4398 m per revolution, which is the circumference of the old 140 mm wheels
and came from the stale URDF. Against the built 120 mm wheels that overstates
speed and distance by 16.7%, so a 0.2 m/s target needs 3395 counts/s per
wheel rather than 2910.

Longitudinal axle positions remain CAD values; the odometry maths does not
use them.

Co-Authored-By: Claude Opus 5 (1M context) <noreply@anthropic.com>

File: ros2_ws/src/space_description/urdf/space_rover.urdf.xacro (robot description, xacro)
@@ -20,16 +20,19 @@
   <xacro:property name="base_width" value="0.26"/>
   <xacro:property name="base_height" value="0.10"/>
-  <!-- Axle centers measured from the complete CAD STL.
-       wheel_radius is NOT from that CAD: the wheels were changed from 140 mm
-       to 120 mm diameter on the physical rover, so it is set from the build
-       rather than the model. The visual mesh still shows the 140 mm wheels.
-       wheel_y is still the CAD value and disagrees with a tape measurement of
-       the physical track width; it has not been reconciled yet. Anything that
-       converts wheel counts to distance must use these values, not the CAD. -->
+  <!-- Wheel geometry is measured from the built rover, not from the CAD.
+       The wheels were changed from 140 mm to 120 mm diameter, and the
+       measured track width is 225 mm against the CAD's 233 mm. Both values
+       below are the measured ones, because everything that converts wheel
+       counts into distance and heading depends on them: the radius scales
+       distance, and the track width scales every turn. The visual mesh still
+       shows the older 140 mm wheels.
+       Longitudinal axle positions are still CAD values and are not used by
+       the odometry maths. -->
   <xacro:property name="wheel_radius" value="0.060"/>
   <xacro:property name="wheel_width" value="0.040"/>
   <xacro:property name="front_wheel_x" value="0.08375"/>
   <xacro:property name="rear_wheel_x" value="-0.06625"/>
-  <xacro:property name="wheel_y" value="0.11650"/>
+  <!-- Half the measured 225 mm track width, centre to centre. -->
+  <xacro:property name="wheel_y" value="0.11250"/>
   <xacro:property name="wheel_z" value="-0.06400"/>
   <material name="chassis_dark"><color rgba="0.10 0.12 0.14 1.0"/></material>
